File: hardware/thermocouple-breakout.sch (KiCad schematic (older format))
At the start: 10 parts, among them P1 CONN_4, P2 CONN_2, U1 AD594/95, U2 74HCT04

Commit message: Updated to kicad 4.0.2
Parts:
- C1: footprint (none) -> visgence_parts:SM0603_Capa_VIS
- D1, D2: footprint (none) -> LEDs:LED_0603
- P1: footprint (none) -> Connect:bornier4
- P2: footprint (none) -> visgence_parts:PCC-SMP
- R1, R2, R3: footprint (none) -> visgence_parts:SM0603_VIS
- U1: footprint (none) -> Housings_DIP:DIP-14_W7.62mm_LongPads
- U2: footprint (none) -> SMD_Packages:SOIC-14_N
Changed lines of the file:
@@
 LIBS:visgence_parts
 LIBS:thermocouple-breakout-cache
-EELAYER 24 0
+EELAYER 25 0
 EELAYER END
 $Descr USLetter 11000 8500
@@
 F 0 "U1" H 4700 2650 60  0000 C CNN
 F 1 "AD594/95" H 4700 2750 60  0000 C CNN
-F 2 "" H 4700 3000 60  0000 C CNN
+F 2 "Housings_DIP:DIP-14_W7.62mm_LongPads" H 4700 3000 60  0001 C CNN
 F 3 "" H 4700 3000 60  0000 C CNN
 	1    4700 3000
@@
 F 0 "P2" V 3650 4650 40  0000 C CNN
 F 1 "CONN_2" V 3750 4650 40  0000 C CNN
-F 2 "" H 3700 4650 60  0000 C CNN
+F 2 "visgence_parts:PCC-SMP" H 3700 4650 60  0001 C CNN
 F 3 "" H 3700 4650 60  0000 C CNN
 	1    3700 4650
@@
 F 0 "P1" V 2750 1300 50  0000 C CNN
 F 1 "CONN_4" V 2850 1300 50  0000 C CNN
-F 2 "" H 2800 1300 60  0000 C CNN
+F 2 "Connect:bornier4" H 2800 1300 60  0001 C CNN
 F 3 "" H 2800 1300 60  0000 C CNN
 	1    2800 1300
@@
 F 0 "R1" V 4830 1250 40  0000 C CNN
 F 1 "R" V 4757 1251 40  0000 C CNN
-F 2 "" V 4680 1250 30  0000 C CNN
+F 2 "visgence_parts:SM0603_VIS" V 4680 1250 30  0001 C CNN
 F 3 "" H 4750 1250 30  0000 C CNN
 	1    4750 1250
@@
 F 0 "D1" H 6650 2600 50  0000 C CNN
 F 1 "ALARM" H 6650 2400 50  0000 C CNN
-F 2 "" H 6650 2500 60  0000 C CNN
+F 2 "LEDs:LED_0603" H 6650 2500 60  0001 C CNN
 F 3 "" H 6650 2500 60  0000 C CNN
 	1    6650 2500
@@
 F 0 "U2" H 5950 1650 40  0000 C CNN
 F 1 "74HCT04" H 6000 1450 40  0000 C CNN
-F 2 "" H 5800 1550 60  0000 C CNN
+F 2 "SMD_Packages:SOIC-14_N" H 5800 1550 60  0001 C CNN
 F 3 "" H 5800 1550 60  0000 C CNN
 	1    5800 1550
@@
 F 0 "R2" V 6730 2000 40  0000 C CNN
 F 1 "1k" V 6657 2001 40  0000 C CNN
-F 2 "" V 6580 2000 30  0000 C CNN
+F 2 "visgence_parts:SM0603_VIS" V 6580 2000 30  0001 C CNN
 F 3 "" H 6650 2000 30  0000 C CNN
 	1    6650 2000
@@
 F 0 "U2" H 7550 1650 40  0000 C CNN
 F 1 "74HCT04" H 7600 1450 40  0000 C CNN
-F 2 "" H 7400 1550 60  0000 C CNN
+F 2 "SMD_Packages:SOIC-14_N" H 7400 1550 60  0001 C CNN
 F 3 "" H 7400 1550 60  0000 C CNN
 	2    7400 1550
@@
 F 0 "U2" H 8550 1650 40  0000 C CNN
 F 1 "74HCT04" H 8600 1450 40  0000 C CNN
-F 2 "" H 8400 1550 60  0000 C CNN
+F 2 "SMD_Packages:SOIC-14_N" H 8400 1550 60  0001 C CNN
 F 3 "" H 8400 1550 60  0000 C CNN
 	3    8400 1550
@@
 F 0 "D2" H 3300 3300 50  0000 C CNN
 F 1 "PWR" H 3300 3100 50  0000 C CNN
-F 2 "" H 3300 3200 60  0000 C CNN
+F 2 "LEDs:LED_0603" H 3300 3200 60  0001 C CNN
 F 3 "" H 3300 3200 60  0000 C CNN
 	1    3300 3200
@@
 F 0 "R3" V 3380 2650 40  0000 C CNN
 F 1 "1k" V 3307 2651 40  0000 C CNN
-F 2 "" V 3230 2650 30  0000 C CNN
+F 2 "visgence_parts:SM0603_VIS" V 3230 2650 30  0001 C CNN
 F 3 "" H 3300 2650 30  0000 C CNN
 	1    3300 2650
@@
 F 0 "C1" H 3600 3050 40  0000 L CNN
 F 1 "C" H 3606 2865 40  0000 L CNN
-F 2 "" H 3638 2800 30  0000 C CNN
+F 2 "visgence_parts:SM0603_Capa_VIS" H 3638 2800 30  0001 C CNN
 F 3 "" H 3600 2950 60  0000 C CNN
 	1    3600 2950
@@
 	6650 2250 6650 2300
 $Comp
-L GND #PWR?
+L GND #PWR012
 U 1 1 531FEB15
 P 4950 4200
-F 0 "#PWR?" H 4950 4200 30  0001 C CNN
+F 0 "#PWR012" H 4950 4200 30  0001 C CNN
 F 1 "GND" H 4950 4130 30  0001 C CNN
 F 2 "" H 4950 4200 60  0000 C CNN
